File: ruuvitracker_kicad/ruuvitracker.sch (KiCad schematic (older format))
At the start: 109 parts, among them J1 USB_MICRO_B, K1 BATTERY, P3 JTAG, P4 USART, U1 STM32F10XXX_LQFP64, U10 TPS799XX, U2 SIM908, U3 LSM303DLHC, U5 MICROPHONE, U6 ESDA6V1W5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

Commit message: Added some logic to detect Micro-USB charger properly + some minor bug fixes.
Parts:
- removed C23: 100u, symbol CAPAPOL
- removed C32: 10u, symbol C
- added C23: 100u, symbol CP1
- added C32: 10u, symbol CP1
- added C42: 100n, symbol C
- added Q1: MOSFET_P, symbol MOSFET_P
- added R48: NA, symbol R
- added R5: 0, symbol R
- added U11: SN74LVC1G38_NAND, symbol SN74LVC1G38_NAND
- C20: value 22p -> 33p
- R1, R2, R4: value 1k -> 10k
- R3: value 0 -> 10k
- R47: renamed from R?; value 100k -> 10k
- gave numbers to parts that had none: 9
Connections:
- net labels added: FLAG1, FLAG2, GSM_CHARGER, SD_CARD_INSERTED
- wire segments 323 -> 341
- no-connect marks 48 -> 41
Other:
- note added: "* Charger connected (D+ and D- shorted) => FLAG1&2 HIGH.\n\n* Over or under voltage (VBUS>6V6 or VBUS < 3V3) => FLAG2 LOW, otherwise HIGH.\n LSCTRL goes HIGH to disable internal PMOS switch."
- note added: "4k7 pull-ups are ok for the SDIO lines."
- note added: "<- If there is no charger detector + NAND gate +\n PMOS assembled, it is possible to connect 5V\n directly to GSM module's VCHG pin."
- note added: "Compatible LQFP64 MCUs:\n\nSTM32F100xx (no USB)\nSTM32F103xx\nSTM32F205xx (only OTG HS)\nSTM32F215xx (only OTG HS)\nSTM32F217xx\nSTM32F405xx\nSTM32F407xx\n\nWhat we want to use:\nSTM32F103RET6\n(512KB flash + 64KB RAM)"
- note added: "Fixed Voltage LDO Regulator"
- note added: "If STM32F20xxx is used and USB cable\nis attached, PA9 = OTG_FS_VBUS = 5V.\n\n(USB OTG device-only connection)"
- note added: "Micro-USB Charger Detection"
- note added: "Open Source Tracking Solution"
- note added: "Optional super capacitor /\nnon-rechargeable battery"
- note added: "REVA"
- note added: "RuuviTracker"
- note added: "Short GPS-VANT-OUT and GPS-VANT-IN\nto apply 2V8 for the active GPS antenna."
- note added: "http://www.ruuvipenkki.fi/ruuvitracker"
- note removed: "* Charger connected (D+ and D- shorted) => FLAG1 HIGH, otherwise LOW.\n\n* Over or under voltage (VBUS>6V6 or VBUS < 3V3) => FLAG2 LOW, otherwise HIGH.\n LSCTRL goes HIGH to disable internal PMOS switch."
- note removed: "4k7 pull-ups are suitable for the SDIO lines."
- note removed: "?"
- note removed: "Compatible LQFP64 MCUs:\n\nSTM32F100xx (no USB)\nSTM32F103xx\nSTM32F205xx (only OTG HS)\nSTM32F215xx (only OTG HS)\nSTM32F217xx\nSTM32F405xx\nSTM32F407xx"
- note removed: "Fixed voltage LDO Regulator"
- note removed: "If STM32F20xxx is used and USB cable\nis attached, PA9 = OTG_FS_VBUS = 5V.\n\n(USB OTG FS (full speed) device-only connection)"
- note removed: "Laturi pitäisi huomata ja syöttää vasta sitten GSM-moduulille laturipinniin virtaa.\n\nVaihtoehtoja detektoripiireiksi:\n\nSTM: STUSBCD01B\nFairchield: FAN3989\n"
- note removed: "RuuviTracker\n REVA"
- moved on the sheet: C1, C10, C11, C12, C13, C14, C15, C16, C17, C18, C19, C2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

Commit message: Some fixes to schematic, created new footprints and .brd file.
Fixed:
- Mirrored MicroSD schematic component

Created:
- Over 10 new footprints
- .cmp file
- .brd file
Parts:
- C10, C9: value 2u2 -> NA
- R22, R23: value 4k7 -> 10k
Connections:
- wire segments 341 -> 343
Other:
- note added: "* Charger connected (D+ and D- shorted) => FLAG1&2 HIGH.\n* Over or under voltage (VBUS>6V6 or VBUS < 3V3) LSCTRL goes HIGH to disable internal PMOS switch."
- note added: "C9,C10,R9 and R10 are for\nmaintaining compability\nbetween STM32F1xx, STM32F2xx\nand STM32F4xx microcontrollers.\n\nLeave R9 and R10 unpopulated if\nF2xx or F4xx series MCU is used.\n\nC9 (2u2) and C10 (2u2) are not needed (but doesn't do\nany harm either) if F1xx series MCU is used.\n\nHowever, the C9 and C10 should not be connected\nwhen the voltage regulator is turned OFF\n(one usecase of F2x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"
- note added: "Compatible holders:\n\n* GCT's MES3051\n* Cheap Chinese version"
- note added: "FLAG1&2 = 0-5V -> STM32's pins need to be 5V tolerant!"
- note added: "Inserting MicroSD card shorts SW-A to SW-B\nie. SD_CARD_INSERTED goes low (IPU required)."
- note added: "Route MIC's signal wires according\ndifferential signal design rules.\n\nPlace capacitors + ESD IC close\nto the microphone."
- note removed: "* Charger connected (D+ and D- shorted) => FLAG1&2 HIGH.\n\n* Over or under voltage (VBUS>6V6 or VBUS < 3V3) => FLAG2 LOW, otherwise HIGH.\n LSCTRL goes HIGH to disable internal PMOS switch."
- note removed: "C9,C10,R9 and R10 are for\nmaintaining compability\nbetween STM32F1xx, STM32F2xx\nand STM32F4xx microcontrollers.\n\nLeave R9 and R10 unpopulated if\nF2xx or F4xx series MCU is used.\n\nC9 and C10 are not needed (but doesn't do\nany harm either) if F1xx series MCU is used.\n\nHowever, the C9 and C10 should not be connected\nwhen the voltage regulator is turned OFF\n(one usecase of F2xx/F4xx MCU)."
- note removed: "Route MIC's signal wires according\ndifferential signal design rules.\n\nPlace capacitors + ESD IC close\nto the microphone(s)."
- moved on the sheet: C24, C33, R31, R32, R33, R34, R35, R36, R37, R38, R39, R40
