File: ruuvitracker_kicad/ruuvitracker.sch (KiCad schematic (older format))
At the start: 114 parts, among them J1 USB_MICRO_B, K1 BATTERY, P1 EXPANDER, P3 JTAG, P4 USART, Q1 MOSFET_P, U1 STM32F10XXX_LQFP64, U10 TPS799XX, U11 SN74LVC1G38_NAND, U2 SIM908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

Commit message: Added two 3mm holes. No routing done yet. Component placement almost ok.
Parts:
- added P2, P5: HOLE, symbol CONN_1
Connections:
- wire segments 343 -> 347
Other:
- note added: "Plated holes"

Commit message: Almost all traces routed. Still 2-layer board, jei! :-)
Connections:
- wire segments 347 -> 348

Commit message: Modified component references on PCB (better alignment).
Parts:
- C41: value 10u -> 4u7
- R12, R18, R19, R6: value 680 -> 330
Connections:
- wire segments 348 -> 436
Other:
- note added: "Plated Holes"
- note added: "REVA 10"
- note added: "Route speaker's signal wires according\ndifferential signal design rules.\n\nPlace capacitors + ESD IC close\nto the speaker."
- note added: "Serial wire JTAG debug port (SWJ-DP) pins:\nJTAG_TMS = SWDIO\nJTAG_TCK = SWCLK"
- note removed: "Plated holes"
- note removed: "REVA"
- note removed: "Route speaker's signal wires according\ndifferential signal design rules.\n\nPlace capacitors + ESD IC\nclose to the speaker."
