File: ruuvitracker_revb_kicad/ruuvitracker.sch (KiCad schematic (older format))
At the start: 117 parts, among them J1 USB_MICRO_B, K1 BATTERY, P2 HOLE, P3 JTAG, P4 USART, P5 HOLE, U2 SIM908, U3 LSM303DLHC, U5 MICROPHONE, U8 MICROSD_SIM_COMBO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

Commit message: New pwr switch and expander connector
Parts:
- removed P?: PWR_SW, symbol CONN_2
- added P?: EXPANDER_HEAD, symbol CONN_18
- added P?: PWR_SW, symbol CONN_3
Connections:
- wire segments 375 -> 457
Other:
- note added: "1 2 3"
- note added: "Alps SSSS811101"
- moved on the sheet: C38, P?, R?

Commit message: Remove speaker's and mic's caps to save space
Parts:
- removed C13, C16, C18, C25, C27, C29: 10p, symbol C
- removed C14, C17, C19, C26, C28, C30: 33p, symbol C
- removed P?: PWR_SW, symbol CONN_3
- added P?: PWR_SW, symbol CONN_4
- P?: value EXPANDER_HEAD -> EXPANDER_3
- R?: value 100k -> 10k
Connections:
- wire segments 457 -> 352
Other:
- note added: "GSM's Microphone"
- note added: "GSM's Speaker"
- note added: "Ground terminals ->"
- note added: "Optional super capacitor /\n3V non-rechargeable battery.\n\nCurrent consumption 2uA after VBAT is removed.\n\nDon't leave unconnected. If not used, populate\n10uF ceramic capacitor for example.\n\n10uF discharging time from 2V8 to\n1V8 @ 2uA = approx. 5 seconds.\n(10mF super cap = approx. one hour)"
- note added: "Place tantalums +\nsmaller ceramic caps close\nto VBAT pins.\n\nMax drawn current during TX\nburst = up to 2A.\n\nReset voltage = 3V1."
- note added: "Route MIC's signal wires according\ndifferential signal design rules.\n\nTrace width should be 6-8 mil.\n\nPlace ESD IC close\nto the microphone."
- note added: "Route speaker's signal wires according\ndifferential signal design rules.\n\nTrace width should be 10-12 mil.\n\nPlace ESD IC close\nto the speaker."
- note removed: "<- Optional amp IC\nshould be placed here"
- note removed: "Microphone"
- note removed: "Optional super capacitor /\n3V non-rechargeable battery.\n\nCurrent consumption 2uA after VBAT is removed.\n\nDon't leave unconnected. If not used, populate\n10uF ceramic capacitor for example."
- note removed: "Place tantalum +\nsmaller ceramic caps close\nto VBAT pins.\n\nMax drawn current during TX\nburst = up to 2A.\n\nReset voltage = 3V1."
- note removed: "Route MIC's signal wires according\ndifferential signal design rules.\n\nTrace width should be 6-8 mil.\n\nPlace capacitors + ESD IC close\nto the microphone."
- note removed: "Route speaker's signal wires according\ndifferential signal design rules.\n\nTrace width should be 10-12 mil.\n\nPlace capacitors + ESD IC close\nto the speaker."
- note removed: "Speaker"
- moved on the sheet: C32, C42, C?, D?, FB1, J1, K1, L?, P?, R21, R25, R28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

Commit message: Add external audio amp
Parts:
- added C? (x2): 1u, symbol C
- added R?: 10k, symbol R
- added U?: LM4890M_MM, symbol LM4890M_MM
Connections:
- net labels added: AUDIO_AMP_SHUTDOWN
- wire segments 352 -> 430
Other:
- note added: "Texas Instruments LM4890MM/NOPB's (MSOP package) key features:\n\n- PSRR at 217Hz, VDD = 5V (Fig. 1) 62 dB(typ.)\n- Power Output at 5V & 1% THD 1 W(typ.)\n- Power Output at 3V3 & 1% THD 400 mW(typ.)\n- Shutdown Current 0.1 μA(typ.)"
- moved on the sheet: SP1

Commit message: Minor mods
Parts:
- removed R25, R28: 22, symbol R
- added RP?: 22, symbol R_PACK4
Connections:
- net labels added: GSM_LINE_IN, GSM_PWRKEY, SPK_AMP_OUT1, SPK_AMP_OUT2
- net labels removed: DCD, DTR, PWRKEY, RING, USART2_RX, USART2_TX, USART3_CTS, USART3_RTS, USART3_RX, USART3_TX
- wire segments 430 -> 362
Other:
- note added: "ESD Protection"
- note added: "Inserting MicroSD card shorts SW-A and SW-B\nie. SD_CARD_INSERTED goes low (IPU required)."
- note added: "Place bypass capacitors +\nESD (TVS) protection ICs\nclose to the card holder."
- note added: "Route speaker's signal wires according\ndifferential signal design rules.\n\nTrace width should be 10-12 mil.\n\nPlace ESD IC close to the speaker."
- note added: "Texas Instruments LM4890MM/NOPB's (MSOP package) key features:\n\n- PSRR at 217Hz, VDD = 5V (Fig. 1) 62 dB (typ.)\n- Power Output at 5V & 1% THD 1 W (typ.)\n- Power Output at 3V3 & 1% THD 400 mW(typ.)\n- Shutdown Current 0.1 μA(typ.)"
- note removed: "ESD Protection\n(MIC + Speaker + SIM)"
- note removed: "Inserting MicroSD card shorts SW-A to SW-B\nie. SD_CARD_INSERTED goes low (IPU required)."
- note removed: "Place bypass capacitors +\nSIM's ESD (TVS) protection array\nclose to the card holder."
- note removed: "Route speaker's signal wires according\ndifferential signal design rules.\n\nTrace width should be 10-12 mil.\n\nPlace ESD IC close\nto the speaker."
- note removed: "Texas Instruments LM4890MM/NOPB's (MSOP package) key features:\n\n- PSRR at 217Hz, VDD = 5V (Fig. 1) 62 dB(typ.)\n- Power Output at 5V & 1% THD 1 W(typ.)\n- Power Output at 3V3 & 1% THD 400 mW(typ.)\n- Shutdown Current 0.1 μA(typ.)"
- moved on the sheet: C11, C12, C24, C33, C34, C35, C36, C38, C40, C41, C?, D1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

Commit message: Minor mods
Parts:
- removed RP? (x2): 4k7, symbol R_PACK4
- removed RP? (x2): 22, symbol R_PACK4
- added R? (x7): 4k7, symbol R
- added R? (x5): 22, symbol R
- C22, C32, C36, C42, C? (x2): value 10u -> 4u7
- C33, C38, C40: value 1u -> 4u7
- D?: value LED -> LED_R
- R2, R? (x6): value 10k -> 4k7
Connections:
- net labels added: ETH_MDC, ETH_RMII_RX_D0, ETH_RMII_RX_D1, ETH_RMII_TXD0, ETH_RMII_TXD1, ETH_RMII_TX_EN, MEMS_MIC_POWER
- net labels removed: GSM_ANT, VBAT
- wire segments 362 -> 429
- no-connect marks 45 -> 41
Other:
- note added: "28 + 18 + 28 = 76 pins total"
- note added: "Current consumption in normal mode 110 μA (typical, magnetic sensor setting ODR = 7.5 Hz, Accelerometer sensor ODR = 50 Hz)\nCurrent consumption in sleep-mode 1 μA (typical, linear accelerometer in sleep-mode and magnetic sensor in power-down mode)"
- note added: "System load delivers all the current (up to 5A) for the system.\nVoltage never drops below 3V5 (programmable) unless battery dies totally."
- note added: "The ADMP404 consists of a MEMS microphone element, an impedance\nconverter, and an output amplifier. The ADMP404 sensitivity specification\nmakes it an excellent choice for both near field and far field applications.\n\nA DC-blocking capacitor is required at the output of the microphone.\nThis capacitor creates a high-pass filter with a corner frequency at\n\nfC = 1/(2π × C × R),\n\nwhere R is th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"
- note removed: "A DC-blocking capacitor is required at the output of the microphone.\nThis capacitor creates a high-pass filter with a corner frequency at\n\nfC = 1/(2π × C × R),\n\nwhere R is the input impedance of the uC's ADC pin.\n\n- Microphone's output impedance = 200ohm.\n- uC ADC's typical input impedance = 6kohm."
- note removed: "Add ADC & DAC pins to IO port!"
- note removed: "System load delivers all the current (up to 5A) for the system.\nVoltage never drops below 3V5 unless battery dies totally."
- moved on the sheet: C42, C6, C7, C?, D?, FB?, K1, L?, R?, U?

Commit message: New USB OTG EMI protection IC
Parts:
- removed R21: 2k2, symbol R
- removed R? (x2): 22, symbol R
- removed U9: TPD2S017, symbol TPD2S017
- added U?: EMIF02-USB04F3, symbol EMIF02-USB04F3
- FB1: value FILTER -> 2A+
Connections:
- net GND: now also U?.B2
- net OTG_FS_ID: now also U?.A1
- net OTG_FS_VBUS: now also FB1.2
- net USB_DM: now also U?.A3
- net USB_DP: now also U?.C3
- net at J1.2 (D-): now also U?.B1
- net at J1.3 (D+): now also U?.C1
- new net PULL_DOWN_TO_ACT_AS_A_HOST: U?.A2, U?.C2
- new net PULL_UP_TO_ACT_AS_A_FS_DEVICE: U?.B3
Other:
- note added: "For best performance, VBUS should be\ndecoupled to PGND with 1μF capacitance."
- note added: "Iinmax = (1V/Rilim)*530\n\nThe actual input current limit is the lower value between ILIM setting and\n register setting (REG00[2:0]). For example, if the register setting is 111\nfor 3A, and ILIM has a 353Ω resistor to ground for 1.5A, the input current\nlimit is 1.5A. ILIM pin can be used to set the input current limit rather than\nthe register settings."
- note added: "Micro-USB-AB + EMI Protection"
- note removed: "EMIF02-USB03F2 olisi ok vaihtoehto, mutta die-size-kotelointi\narvelluttaa ja lisäksi sitä ei ole saatavilla Mouser/DK... STM:llä\nei vastaavia OTG:lle suunniteltuja..."
- note removed: "For best performance, VBUS should be\ndecoupleto PGND with 1μF capacitance."
- note removed: "Micro-USB-AB"
- moved on the sheet: FB1, J1, P?

Commit message: USB ESD modifications
Parts:
- removed U?: EMIF02-USB04F3, symbol EMIF02-USB04F3
- added JP?: JUMPER, symbol JUMPER
- added R? (x2): 22, symbol R
- added U?: TPD2S017, symbol TPD2S017
Connections:
- net GND: now also U?.2 (GND)
- net OTG_FS_VBUS: now also JP?.2, U?.5 (VCC); no longer U?.1 (VBUS), U?.24 (VBUS)
- net USB_DM: now also R?.2
- net USB_DP: now also R?.1
- net at FB1.1, J1.1 (VBUS): no longer P?.1 (P1)
- net at J1.2 (D-): now also U?.3 (CH1In)
- net at J1.3 (D+): now also U?.4 (CH2Int)
- new net: R?.1, U?.1 (CH1Out)
- new net: R?.2, U?.6 (CH2Out)
- new net HIGH_VOLTAGE_VBUS: JP?.1, P?.1 (P1), U?.1 (VBUS), U?.24 (VBUS)
Other:
- note added: "If using over 5V power sources (17VDC max), remove\nsolder bridge to save the ARM's life!\nUSB (device mode) is still functioning, but OTG is disabled."
- note added: "Micro-USB-AB + ESD Protection"
- note removed: "Micro-USB-AB + EMI Protection"
- moved on the sheet: FB1, J1, P?

Commit message: Minor mods
Parts:
- removed C20: 33p, symbol C
- removed JP?: JUMPER, symbol JUMPER
- added R?: 0, symbol R
Connections:
- net DAC_OUT1 is gone; now on net GSM_LINE_IN: C31.2
- net HIGH_VOLTAGE_VBUS: now also R?.1
- net OTG_FS_VBUS: now also R?.2
- net GPS_ANT: no longer names the net of U2.79 (GPS-ANT)
- no-connect marks 41 -> 42
Other:
- note added: "If using over 5V power sources (17VDC max), remove\nzero ohm resistor to save the ARM's life!\n\nUSB (device mode) is still functioning, but OTG\ncannot be used."
- note removed: "If using over 5V power sources (17VDC max), remove\nsolder bridge to save the ARM's life!\nUSB (device mode) is still functioning, but OTG is disabled."
- moved on the sheet: P?, R?
Changed lines of the file:
@@
-EESchema Schematic File Version 2  date Thu 20 Dec 2012 12:37:29 PM EET
+EESchema Schematic File Version 2  date Fri 21 Dec 2012 01:29:10 AM EET
 LIBS:power
 LIBS:device
@@
 Comment4 ""
 $EndDescr
+NoConn ~ 26900 7900
+Wire Wire Line
+	-300 13600 -450 13600
+Wire Wire Line
+	-1500 14450 -1400 14450
 Wire Wire Line
 	16550 30450 16550 30550
 Wire Wire Line
-	16400 32050 16500 32050
+	-650 12600 -550 12600
 Wire Wire Line
-	16500 32050 16500 32150
+	-550 12600 -550 12700
 Wire Wire Line
 	17750 30900 17650 30900
@@
 	14800 30550 14900 30550
 Wire Wire Line
-	-450 13600 -350 13600
-Wire Wire Line
 	15400 31250 15500 31250
 Wire Wire Line
@@
 	7100 20550 7100 21250
 Wire Wire Line
-	-550 13750 -550 13850
-Wire Wire Line
 	28500 26850 28150 26850
 Wire Wire Line
@@
 	7600 29700 7500 29700
 Wire Wire Line
-	23650 28300 23450 28300
+	23450 28300 23650 28300
 Connection ~ 23550 28000
 Wire Wire Line
@@
 	6500 20450 6450 20500
 Wire Wire Line
-	-4800 27950 -5000 27950
+	-5000 27950 -4800 27950
 Wire Wire Line
 	-4800 27850 -4900 27850
@@
 	16600 10000 16500 10000
 Wire Wire Line
-	16800 8150 16400 8150
+	16400 8150 16800 8150
 Wire Wire Line
 	16750 12150 16750 12050
@@
 	16400 13950 16500 13950
 Wire Wire Line
-	15550 28050 14900 28050
+	14900 28050 15550 28050
 Wire Wire Line
 	15200 28650 15200 28600
@@
 	32200 28400 32100 28400
 Wire Wire Line
-	23000 9500 23100 9500
+	23000 9500 23400 9500
 Wire Wire Line
-	23600 9600 24500 9600
+	23900 9600 24500 9600
 Wire Wire Line
-	24500 9400 23600 9400
+	24500 9400 23900 9400
 Wire Wire Line
 	23100 9200 24500 9200
@@
 	-1500 28450 -1500 28550
 Wire Wire Line
-	-1500 27800 -1500 28050
+	-1500 28050 -1500 27800
 Wire Wire Line
-	-300 27800 -300 28050
+	-300 28050 -300 27800
 Wire Wire Line
 	10300 22200 10200 22200
@@
 Wire Wire Line
 	29750 13200 29850 13200
-Connection ~ 23800 9400
-Wire Wire Line
-	23800 9650 23800 9400
 Wire Wire Line
 	27250 12100 27250 12050
@@
 	27250 11600 26900 11600
 Wire Wire Line
-	23800 10100 23800 10050
-Wire Wire Line
 	5500 28050 5500 27800
 Connection ~ 5500 27800
@@
 	28300 27100 28500 27100
 Wire Wire Line
-	26400 12500 25600 12500
+	25600 12500 26400 12500
 Connection ~ 25700 12500
 Wire Wire Line
-	6100 27800 5300 27800
+	5300 27800 6100 27800
 Connection ~ 32850 28200
 Connection ~ 32850 28400
@@
 	34700 27100 35250 27100
 Wire Wire Line
-	23600 9500 24500 9500
+	23900 9500 24500 9500
 Wire Wire Line
-	23000 9600 23100 9600
+	23000 9600 23400 9600
 Wire Wire Line
-	23000 9400 23100 9400
+	23000 9400 23400 9400
 Wire Wire Line
 	32200 28500 32100 28500
@@
 	6100 28000 6000 28000
 Wire Wire Line
-	8250 27700 8250 28150
+	8250 28150 8250 27700
 Connection ~ 8250 27800
 Wire Wire Line
-	14300 27850 15550 27850
+	15550 27850 14300 27850
 Wire Wire Line
 	14950 28650 14950 28600
@@
 	350  15350 450  15350
 Connection ~ 350  15350
-Wire Wire Line
-	250  13600 350  13600
 Connection ~ 350  13600
 Wire Wire Line
@@
 	-450 14900 -250 14900
 Wire Wire Line
-	250  14900 450  14900
+	450  14900 250  14900
 Wire Wire Line
 	-950 14900 -850 14900
@@
 	16500 10000 16500 9900
 Wire Wire Line
-	16800 8400 16500 8400
+	16500 8400 16800 8400
 Connection ~ 16600 8400
 Wire Wire Line
@@
 Wire Wire Line
 	28150 27850 28150 27800
-Wire Wire Line
-	450  14450 -550 14450
-Wire Wire Line
-	-550 14450 -550 14350
 Wire Notes Line
 	6400 20550 6400 21250
@@
 	6550 20400 6950 20400
 Wire Wire Line
-	17150 11550 16400 11550
+	16400 11550 17150 11550
 Wire Wire Line
 	32850 28700 32850 28050
@@
 Wire Wire Line
 	16550 31550 16550 31450
+Wire Wire Line
+	-900 14450 450  14450
+Wire Wire Line
+	200  13600 350  13600
+$Comp
+L R R?
+U 1 1 50D39DBF
+P -50 13600
+F 0 "R?" V 30  13600 50  0000 C CNN
+F 1 "0" V -50 13600 50  0000 C CNN
+	1    -50  13600
+	0    1    1    0
+$EndComp
+Text Label 25100 12500 2    60   ~ 0
+GSM_LINE_IN
 Text Label 16550 30450 2    60   ~ 0
 OTG_FS_VBUS
@@
 	1    0    0    -1
 $EndComp
-$Comp
-L JUMPER JP?
-U 1 1 50D2E8A9
-P -50 13600
-F 0 "JP?" H -50 13750 60  0000 C CNN
-F 1 "JUMPER" H -50 13520 40  0000 C CNN
-	1    -50  13600
-	-1   0    0    1
-$EndComp
-Text Label 16400 31850 0    60   ~ 0
+Text Label -650 12400 0    60   ~ 0
 HIGH_VOLTAGE_VBUS
 Text Label -450 13450 2    60   ~ 0
@@
 Text Label 29150 14250 2    60   ~ 0
 OTG_FS_ID
-Text Notes -1500 13150 0    40   Italic 0
-If using over 5V power sources (17VDC max), remove\nsolder bridge to save the ARM's life!\nUSB (device mode) is still functioning, but OTG is disabled.
+Text Notes -1450 13050 0    40   Italic 0
+If using over 5V power sources (17VDC max), remove\nzero ohm resistor to save the ARM's life!\n\nUSB (device mode) is still functioning, but OTG\ncannot be used.
 Text Label 3850 7300 0    60   ~ 0
 PULL_DOWN_TO_ACT_AS_A_HOST
@@
 L GND #PWR?
 U 1 1 50D0E7B0
-P 16500 32150
-F 0 "#PWR?" H 16500 32150 30  0001 C CNN
-F 1 "GND" H 16500 32080 30  0001 C CNN
-	1    16500 32150
+P -550 12700
+F 0 "#PWR?" H -550 12700 30  0001 C CNN
+F 1 "GND" H -550 12630 30  0001 C CNN
+	1    -550 12700
 	1    0    0    -1
 $EndComp
@@
 L R R?
 U 1 1 50C95765
-P 23350 9600
-F 0 "R?" V 23350 9700 50  0000 C CNN
-F 1 "22" V 23350 9500 50  0000 C CNN
-	1    23350 9600
+P 23650 9600
+F 0 "R?" V 23650 9700 50  0000 C CNN
+F 1 "22" V 23650 9500 50  0000 C CNN
+	1    23650 9600
 	0    -1   -1   0
 $EndComp
@@
 L R R?
 U 1 1 50C95763
-P 23350 9500
-F 0 "R?" V 23350 9600 50  0000 C CNN
-F 1 "22" V 23350 9400 50  0000 C CNN
-	1    23350 9500
+P 23650 9500
+F 0 "R?" V 23650 9600 50  0000 C CNN
+F 1 "22" V 23650 9400 50  0000 C CNN
+	1    23650 9500
 	0    -1   -1   0
 $EndComp
@@
 L R R?
 U 1 1 50C95742
-P 23350 9400
-F 0 "R?" V 23350 9500 50  0000 C CNN
-F 1 "22" V 23350 9300 50  0000 C CNN
-	1    23350 9400
+P 23650 9400
+F 0 "R?" V 23650 9500 50  0000 C CNN
+F 1 "22" V 23650 9300 50  0000 C CNN
+	1    23650 9400
 	0    -1   -1   0
 $EndComp
@@
 L R R?
 U 1 1 5083DAB8
-P -550 14100
-F 0 "R?" V -470 14100 50  0000 C CNN
-F 1 "4k7" V -550 14100 50  0000 C CNN
-	1    -550 14100
-	-1   0    0    1
+P -1150 14450
+F 0 "R?" V -1070 14450 50  0000 C CNN
+F 1 "4k7" V -1150 14450 50  0000 C CNN
+	1    -1150 14450
+	0    1    1    0
 $EndComp
-Text Label -550 13750 2    60   ~ 0
+Text Label -1500 14450 2    60   ~ 0
 SYSTEM_LOAD
 Text Label -950 15050 2    60   ~ 0
@@
 L CONN_2 P?
 U 1 1 50819F4B
-P 16050 31950
-F 0 "P?" V 16000 31950 40  0000 C CNN
-F 1 "PWR" V 16100 31950 40  0000 C CNN
-	1    16050 31950
+P -1000 12500
+F 0 "P?" V -1050 12500 40  0000 C CNN
+F 1 "PWR" V -950 12500 40  0000 C CNN
+	1    -1000 12500
 	-1   0    0    -1
 $EndComp
@@
 	1    0    0    -1
 $EndComp
-Text Label 26900 7900 0    60   ~ 0
-GPS_ANT
 $Comp
 L SMF05C U?
@@
 	0    1    1    0
 $EndComp
-Text Label 25100 12500 2    60   ~ 0
-DAC_OUT1
 Text Notes 26950 29600 2    40   Italic 0
 Electret Condenser Microphone
@@
 	0    1    1    0
 $EndComp
-$Comp
-L GND #PWR048
-U 1 1 4EF8E9DF
-P 23800 10100
-F 0 "#PWR048" H 23800 10100 30  0001 C CNN
-F 1 "GND" H 23800 10030 30  0001 C CNN
-	1    23800 10100
-	-1   0    0    -1
-$EndComp
-$Comp
-L C C20
-U 1 1 4EF8E9D3
-P 23800 9850
-F 0 "C20" H 23850 9950 50  0000 L CNN
-F 1 "33p" H 23850 9750 50  0000 L CNN
-	1    23800 9850
-	1    0    0    -1
-$EndComp
 Text Label 26900 8800 0    60   ~ 0
