File: ruuvitracker_revb_kicad/ruuvitracker.sch (KiCad schematic (older format))
At the start: 116 parts, among them J1 USB_MICRO_B, K1 BATTERY, P2 HOLE, P3 JTAG, P4 USART, P5 HOLE, U2 SIM908, U3 LSM303DLHC, U5 MICROPHONE, U8 MICROSD_SIM_COMBO, X1 4-26MHZ

Commit message: Another ESD IC replacement
Parts:
- removed U? (x4): SMF05C, symbol SMF05C
- removed U?: TPD2S017, symbol TPD2S017
- added C? (x5): 100n, symbol C
- added U? (x5): TPD4E004, symbol TPD4E004
Connections:
- wire segments 365 -> 450
- no-connect marks 42 -> 40
Other:
- moved on the sheet: R?

Commit message: Minor mods
Parts:
- added C?: 100n, symbol C
- added C?: 10p, symbol C
- added P?: SPK_BEFORE_AMP, symbol CONN_2
- added P? (x2): HOLE, symbol CONN_1
- added U?: TPD4E004, symbol TPD4E004
Connections:
- net labels added: GSM_NETLIGHT, GSM_STATUS
- net labels removed: GSM_NETLIGHT_LED, GSM_STATUS_LED
- wire segments 450 -> 403
- no-connect marks 40 -> 45
Other:
- note added: "Fiducials"
- note added: "IO Pins' absolute maximum voltage = 3V1\nHigh level voltage = 2V8\nMaximum xurrent = 10mA\n"
- note added: "Leave copper keep-out area under the GSM and GPS antenna pins (pins 59 and 79)."
- note removed: "IO Pins' absolute maximum voltage = 3V1.\nIO Pins' high level voltage == 2V8."
- moved on the sheet: C?

Commit message: Add testpoints
Parts:
- added P? (x8): TP, symbol TP
- added R? (x6): 1k, symbol R
- C?: value 100u -> 470u
- FB1: value 2A+ -> FILTER
- R1: value 10k -> 4k7
Connections:
- net labels added: GSM_MIC1N, GSM_MIC1P, GSM_MIC2N, GSM_MIC2P, GSM_SPK1N, GSM_SPK1P
- net labels removed: MIC1N, MIC1P, MIC2N, MIC2P, SPK1N, SPK1P
- wire segments 403 -> 418
Other:
- note added: "Input\nto the\nmodule"
- note added: "Output\nfrom the\nmodule\n(2V8 level)"
- note added: "Reference design uses 22pF cap on data line."
- note removed: "Input to the module"
- note removed: "Output from the module"
- moved on the sheet: C?, P?, R?, U5

Commit message: New level-shifter IC
Parts:
- added C? (x2): 100n, symbol C
- added U?: SN74AVC4T245_RSV, symbol SN74AVC4T245_RSV
Connections:
- net labels added: GPS/DBG-RXD_3V3SIDE, GSM_CTS_3V3SIDE, GSM_DTR_3V3SIDE, GSM_RXD_3V3SIDE
- wire segments 418 -> 432
Other:
- note added: "A PORT\nEnabled\nHi-Z\nHi-Z"
- note added: "B PORT\nHi-Z\nEnabled\nHi-Z"
- note added: "CONTROL INPUTS"
- note added: "DIR\nL\nH\nX"
- note added: "OPERATION"
- note added: "OUTPUT CIRCUITS"
- note added: "SN74AVC4T245RSVR (SN74AVCH4T245RSVR is pin and function compatible)"
- note added: "\nB data to A bus\nA data to B bus\nIsolation"
- note added: "~OE\nL\nL\nH"
- moved on the sheet: C11, C12, C24, C33, C?, D1, D2, D3, D4, D?, FB1, J1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

Commit message: New buttons
Parts:
- removed P?: BOOT0, symbol CONN_2
- removed SW? (x3): SW_PUSH, symbol SW_PUSH
- added R?: 4k7, symbol R
- added SW? (x2): PUSH_BUTTON, symbol PUSH_BUTTON
- C32: value 4u7 -> SUPERCAP
- R20: value 2k2 -> 1k
Connections:
- net labels added: USER_BUTTON
- net labels removed: 1ST_USER_BUTTON, 2ND_USER_BUTTON, 3RD_USER_BUTTON, PULL_DOWN_TO_ACT_AS_A_HOST, PULL_UP_TO_ACT_AS_A_FS_DEVICE
- wire segments 432 -> 442
- no-connect marks 45 -> 43
Other:
- note added: "Alps SKSGPAE010"
- note added: "GSM / GPS Module"
- note added: "LINE-IN input range (peak-to-peak) <500mV!"
- note added: "Outputs\nfrom the\nmodule\n(2V8 level)"
- note added: "Place tantalums +\nsmaller ceramic caps close\nto VBAT pins.\n\nMax drawn current during TX\nburst = up to 2A.\n\nReset voltage level = 3V1."
- note added: "R is used to adjust bias voltage level (1uF and 1kohm produce 1V5 bias voltage level).\nFor more information, please refer application note AN_SIM900_Audio_LINE-IN_Input."
- note added: "Short GPS-VANT-OUT and GPS-VANT-IN using zero\nohm resistor to apply 2V8 for the active GPS antenna."
- note added: "Some SW debouncing\nmight be needed."
- note removed: "GSM / GPRS / GPS Module"
- note removed: "If used, button pins require internal\npull-downs set on from the software."
- note removed: "Input\nto the\nmodule"
- note removed: "Place tantalums +\nsmaller ceramic caps close\nto VBAT pins.\n\nMax drawn current during TX\nburst = up to 2A.\n\nReset voltage = 3V1."
- note removed: "R is used to adjust bias voltage level.\nFor more information, please refer application\nnote AN_SIM900_Audio_LINE-IN_Input."
- note removed: "Short GPS-VANT-OUT and GPS-VANT-IN\nto apply 2V8 for the active GPS antenna."
- moved on the sheet: C21, C22, C23, C31, C?, R20, U?

Commit message: Some thinking about pinouts
Connections:
- net ACCMAGN_INT2: no longer U?.24 (PA1-USART2_RTS/UART4_RX/ETH_RMII_REF_CLK/ETH_MII_RX_CLK/TIM5_CH2/TIMM2_CH2/EVENTOUT-ADC123_IN1)
- net GPS/DBG-RXD_3V3SIDE: now also U?.92 (PB6-I2C1_SCL/TIM4_CH1/CAN2_TX/DCMI_D5/USART1_TX/EVENTOUT); no longer U?.25 (PA2-USART2_TX/TIM5_CH3/TIM9_CH1/TIM2_CH3/ETH_MDIO/EVENTOUT-ADC123_IN2)
- net GPS/DBG-TXD: now also U?.93 (PB7-I2C1_SDA/FSMC_NL/DCMI_VSYNC/USART1_RX/TIM4_CH2/EVENTOUT); no longer U?.26 (PA3-USART2_RX/TIM5_CH4/TIM9_CH2/TIM2_CH4/OTG_HS_ULPI_D0/ETH_MII_COL/EVENTOUT-ADC123_IN3)
- net GSM_CTS_3V3SIDE: now also U?.85 (PD4-FSMC_NOE/USART2_RTS/EVENTOUT); no longer U?.53 (PB14-SPI2_MISO/TIM1_CH2N/TIM12_CH1/OTG_HS_DM/USART3_RTS/TIM8_CH2N/I2S2ext_SD/EVENTOUT)
- net GSM_LINE_IN: now also U?.30 (PA5-SPI1_SCK/OTG_HS_ULPI_CK/TIM2_CH1_ETR/TIM8_CHIN/EVENTOUT-ADC123_IN5/DAC2_OUT); no longer U?.29 (PA4-SPI1_NSS/SPI3_NSS/USART2_CK/DCMI_HSYNC/OTG_HS_SOF/I2S3_WS/EVENTOUT-ADC123_IN4/DAC1_OUT)
- net GSM_RTS: now also U?.84 (PD3-FSMC_CLK/USART2_CTS/EVENTOUT); no longer U?.52 (PB13-SPI2_SCK/I2S2_CK/USART3_CTS/TIM1_CH1N/CAN2_TX/OTG_HS_ULPI_D6/ETH_RMII_TXD1/ETH_MII_TXD1/EVENTOUT-OTG_HS_VBUS)
- net GSM_RXD_3V3SIDE: now also U?.86 (PD5-FSMC_NWE/USART2_TX/EVENTOUT); no longer U?.47 (PB10-SPI2_SCK/I2S2_CK/I2C2_SCL/USART3_TX/OTG_HS_ULPI_D3/ETH_MII_RX_ER/TIM2_CH3/EVENTOUT)
- net GSM_TXD: now also U?.87 (PD6-FSMC_NWAIT/USART2_RX/EVENTOUT); no longer U?.48 (PB11-I2C2_SDA/USART3_RX/OTG_HS_ULPI_D4/ETH_RMII_TX_EN/ETH_MII_TX_EN/TIM2_CH4/EVENTOUT)
- net I2C_SCL: now also U?.95 (PB8-TIM4_CH3/SDIO_D4/TIM10_CH1/DCMI_D6/ETH_MII_TXD3/I2C1_SCL/CAN1_RX/EVENTOUT); no longer U?.92 (PB6-I2C1_SCL/TIM4_CH1/CAN2_TX/DCMI_D5/USART1_TX/EVENTOUT)
- net I2C_SDA: now also U?.96 (PB9-SPI2_NSS/I2S2_WS/TIM4_CH4/TIM11_CH1/SDIO_D5/DCMI_D7/I2C1_SDA/CAN1_TX/EVENTOUT); no longer U?.93 (PB7-I2C1_SDA/FSMC_NL/DCMI_VSYNC/USART1_RX/TIM4_CH2/EVENTOUT)
- net SD_CARD_INSERTED: no longer U?.64 (PC7-I2S3_MCK/TIM8_CH2/SDIO_D7/USART6_RX/DCMI_D1/TIM3_CH2/EVENTOUT)
Other:
- note added: "ETHERNET\nReduced media-independent interface: RMII"
Changed lines of the file:
@@
-EESchema Schematic File Version 2  date Sat 22 Dec 2012 10:51:24 PM EET
+EESchema Schematic File Version 2  date Sun 23 Dec 2012 04:20:00 AM EET
 LIBS:power
 LIBS:device
@@
 Sheet 1 1
 Title "RuuviTracker"
-Date "22 dec 2012"
+Date "23 dec 2012"
 Rev "RevB"
 Comp "RuuviTracker.fi / Lauri Jämsä / lauri.jamsa@ruuvipenkki.fi"
@@
 Comment4 ""
 $EndDescr
+Text Label 8050 10850 2    60   ~ 0
+CAN1_TX
+Text Label 8050 10750 2    60   ~ 0
+CAN1_RX
+Wire Notes Line
+	8050 14100 8050 5400
+Wire Notes Line
+	8600 14100 8600 5400
 Connection ~ 6400 35300
 Wire Wire Line
@@
 	2150 14050 2250 14050
 Wire Wire Line
-	9700 6550 10300 6550
-Wire Wire Line
 	9250 7750 10300 7750
 Wire Wire Line
@@
 	9250 7850 10300 7850
 Wire Wire Line
-	9700 6650 10300 6650
-Wire Wire Line
 	2250 14050 2250 14150
 Wire Wire Line
@@
 Wire Wire Line
 	6400 35500 6300 35500
+Wire Notes Line
+	9300 14100 9300 5400
+Wire Notes Line
+	8750 5400 8750 14100
+Text Label 8050 8550 2    60   ~ 0
+CAN2_RX
+Text Label 8050 8650 2    60   ~ 0
+CAN2_TX
+Text Label 8750 6450 2    60   ~ 0
+MCO1_CONNECTEC_TO_REF_CLK
+Text Label 8750 5750 2    60   ~ 0
+ETH_RMII_REF_CLK
+Text Label 8750 6350 2    60   ~ 0
+ETH_RMII_CRS_DV
+Text Label 8750 5850 2    60   ~ 0
+ETH_MDIO
+Text Notes 8750 5350 1    40   Italic 0
+ETHERNET\nReduced media-independent interface: RMII
 $Comp
 L PUSH_BUTTON SW?
@@
 	1    0    0    -1
 $EndComp
-Text Label 10300 5850 2    60   ~ 0
+Text Label 10300 7950 2    60   ~ 0
 GPS/DBG-RXD_3V3SIDE
-Text Label 10300 8350 2    60   ~ 0
+Text Label 10300 11250 2    60   ~ 0
 GSM_RXD_3V3SIDE
-Text Label 10300 8750 2    60   ~ 0
+Text Label 10300 11150 2    60   ~ 0
 GSM_CTS_3V3SIDE
 Text Label 5400 8800 2    60   ~ 0
@@
 Text Label -450 13450 2    60   ~ 0
 HIGH_VOLTAGE_VBUS
-Text Label 9700 6550 2    60   ~ 0
+Text Label 10300 6550 2    60   ~ 0
 OTG_FS_VBUS
 Text Notes -1450 13050 0    40   Italic 0
@@
 Text Label -450 13600 2    60   ~ 0
 OTG_FS_VBUS
-Text Label 10300 8450 2    60   ~ 0
+Text Label 10300 11350 2    60   ~ 0
 GSM_TXD
-Text Label 10300 8650 2    60   ~ 0
+Text Label 10300 11050 2    60   ~ 0
 GSM_RTS
 Text Label 4950 9100 0    60   ~ 0
@@
 Text Label 4950 9000 0    60   ~ 0
 GSM_DCD
-Text Label 10300 5950 2    60   ~ 0
+Text Label 10300 8050 2    60   ~ 0
 GPS/DBG-TXD
 Text Label 13200 33750 0    60   ~ 0
@@
 Text Label 8600 12450 2    60   ~ 0
 DCMI_D2
-Text Label 8600 6650 2    60   ~ 0
+Text Label 8600 9750 2    60   ~ 0
 DCMI_D1
-Text Label 8600 6550 2    60   ~ 0
+Text Label 8600 9650 2    60   ~ 0
 DCMI_D0
 Text Label 8600 12950 2    60   ~ 0
@@
 Text Label 15550 31500 0    60   ~ 0
 OTG_FS_ID
-Text Label 9700 6650 2    60   ~ 0
+Text Label 10300 6650 2    60   ~ 0
 OTG_FS_ID
 Text Notes 16200 7650 0    30   Italic 0
@@
 	1    0    0    -1
 $EndComp
-Text Label 10300 9750 2    60   ~ 0
+Text Label 5150 9450 2    60   ~ 0
 SD_CARD_INSERTED
 Text Label 18650 35150 2    60   ~ 0
@@
 Text Notes 24000 33750 0    120  Italic 0
 Line-In
-Text Label 10300 6050 2    60   ~ 0
+Text Label 10300 6150 2    60   ~ 0
 GSM_LINE_IN
 $Comp
@@
 	1    0    0    -1
 $EndComp
-Text Label 10300 5750 2    60   ~ 0
+Text Label 4800 7550 2    60   ~ 0
 ACCMAGN_INT2
 Text Label 10300 5650 2    60   ~ 0
@@
 Text Label 28000 9200 0    60   ~ 0
 GSM_RTS
-Text Label 10300 8050 2    60   ~ 0
+Text Label 10300 8250 2    60   ~ 0
 I2C_SDA
-Text Label 10300 7950 2    60   ~ 0
+Text Label 10300 8150 2    60   ~ 0
 I2C_SCL
 $Comp
@@
 Text Label 23000 9200 2    60   ~ 0
 GPS/DBG-TXD
-Text Label 10300 6650 2    60   ~ 0
-USART1_RX
-Text Label 10300 6550 2    60   ~ 0
-USART1_TX
 Text Label 16400 6900 0    60   ~ 0
 STM32_RST

Commit message: Some pin arrangement
Parts:
- added R? (x2): 0, symbol R
Connections:
- net ACCMAGN_DRDY: now also U?.53 (PB14-SPI2_MISO/TIM1_CH2N/TIM12_CH1/OTG_HS_DM/USART3_RTS/TIM8_CH2N/I2S2ext_SD/EVENTOUT)
- net ACCMAGN_INT2: now also U?.36 (PB1-TIM3_CH4/TIM8_CH3N/OTG_HS_ULPI_D2/ETH_MII_RXD3/TIM1_CH3N/EVENTOUT-ADC12_IN9)
- net AUDIO_AMP_SHUTDOWN: now also U?.9 (PC15-EVENTOUT-OSC32_OUT)
- net GPS/DBG-RXD_3V3SIDE: now also R?.1; no longer U?.92 (PB6-I2C1_SCL/TIM4_CH1/CAN2_TX/DCMI_D5/USART1_TX/EVENTOUT)
- net GPS/DBG-TXD: now also R?.1; no longer U?.93 (PB7-I2C1_SDA/FSMC_NL/DCMI_VSYNC/USART1_RX/TIM4_CH2/EVENTOUT)
- net GSM_DCD: now also U?.18 (PC3-SPI2_MOSI/I2S2_SD/OTG_HS_ULPI_NXT/ETH_MII_TX_CLK/EVENTOUT-ADC123_IN13)
- net GSM_DTR_3V3SIDE: now also U?.8 (PC14-EVENTOUT-OSC32_IN)
- net GSM_PWRKEY: now also U?.1 (PE2-TRACECLK/FSMC_A23/ETH_MII_TXD3/EVENTOUT)
- net GSM_RI: now also U?.17 (PC2-SPI2_MISO/OTG_HS_ULPI_DIR/TH_MII_TXD2/I2S2ext_SD/EVENTOUT-ADC123-IN12)
- net HAPTIC_EN: now also U?.7 (PC13-EVENTOUT-RTC_AF1)
- net HAPTIC_PWM: now also U?.54 (PB15-SPI2_MOSI/I2S2_SD/TIM1_CH3N/TIM8_CH3N/TIM12_CH2/OTG_HS_DP/EVENTOUT)
- net LED1: now also U?.58 (PD11-FSMC_CLE/FSMC_A16/USART3_CTS/EVENTOUT)
- net LED2: now also U?.59 (PD12-FSMC_ALE/FSMC_A17/TIM4_CH1/USART3_RTS/EVENTOUT)
- net LED3: now also U?.60 (PD13-FSMC_A18/TIM4_CH2/EVENTOUT)
- net MEMS_MIC_OUTPUT: now also U?.26 (PA3-USART2_RX/TIM5_CH4/TIM9_CH2/TIM2_CH4/OTG_HS_ULPI_D0/ETH_MII_COL/EVENTOUT-ADC123_IN3)
- net MEMS_MIC_POWER: now also U?.35 (PB0-TIM3_CH3/TIM8_CH2N/OTG_HS_ULPI_D1/ETH_MII_RXD2/TIM1_CH2N/EVENTOUT-ADC12_IN8)
- net SD_CARD_INSERTED: now also U?.2 (PE3-TRACED0/FSMC_A19/EVENTOUT)
- net SPI1_MOSI: no longer U?.91 (PB5-I2C1_SMBA/CAN2_RX/OTG_HS_ULPI_D7/ETH_PPS_OUT/TIM3_CH2/SPI1_MOSI/SPI3_MOSI/DCMI_D10/I2S3_SD/EVENTOUT)
- net USER_BUTTON: now also U?.47 (PB10-SPI2_SCK/I2S2_CK/I2C2_SCL/USART3_TX/OTG_HS_ULPI_D3/ETH_MII_RX_ER/TIM2_CH3/EVENTOUT)
- net PC0: now reaches U?.15 (PC0-OTG_HS_ULPI_STP/EVENTOUT-ADC123_IN10)
- net PC0: now also R?.1
- new net PB6: R?.2, U?.92 (PB6-I2C1_SCL/TIM4_CH1/CAN2_TX/DCMI_D5/USART1_TX/EVENTOUT)
- new net PB7: R?.2, U?.93 (PB7-I2C1_SDA/FSMC_NL/DCMI_VSYNC/USART1_RX/TIM4_CH2/EVENTOUT)
Other:
- note added: "<-- Pins to the expansion slot"
- note added: "Route MIC's signal wires according\ndifferential signal design rules.\n\nFor multi-layers PCB, audio lines should be\nlayout in the middle layer, and keep ground\nlayer under audio layer.\n\nTrace width should be 6-8 mil.\n\nPlace ESD IC close to the microphone."
- note removed: "Route MIC's signal wires according\ndifferential signal design rules.\n\nTrace width should be 6-8 mil.\n\nPlace ESD IC close\nto the microphone."
- moved on the sheet: C42, C?, D?, K1, L?, P?, R?, U?

Commit message: Little more pin arrangement
Parts:
- added R? (x2): 4k7, symbol R
- added R?: 0, symbol R
- added R?: 1k, symbol R
- C34: value 220n -> 100n
- D?: value LED_R -> LED_RED
Connections:
- net BATTERY_CELL: now also C?.1; no longer C?.2
- net CHARGER_ENABLE: now also U?.59 (PD12-FSMC_ALE/FSMC_A17/TIM4_CH1/USART3_RTS/EVENTOUT), R?.1
- net CHARGER_INTERRUPT: now also U?.60 (PD13-FSMC_A18/TIM4_CH2/EVENTOUT)
- net CHARGER_STATUS: now also U?.58 (PD11-FSMC_CLE/FSMC_A16/USART3_CTS/EVENTOUT)
- net GND: now also C?.2, R?.1, R?.2; no longer C?.1
- net HIGH_VOLTAGE_VBUS: now also C?.2
- net LED1: now also U?.3 (PE4-TRACED1/FSMC_A20/DCMI_D4/_EVENTOUT); no longer U?.58 (PD11-FSMC_CLE/FSMC_A16/USART3_CTS/EVENTOUT)
- net LED2: now also U?.4 (PE5-TRACED2/FSMC_A21/TIM9_CH1/DCMI_D6/EVENTOUT); no longer U?.59 (PD12-FSMC_ALE/FSMC_A17/TIM4_CH1/USART3_RTS/EVENTOUT)
- net LED3: now also U?.5 (PE6-TRACED3/FSMC_A22/TIM9_CH2/DCMI_D7/EVENTOUT); no longer U?.60 (PD13-FSMC_A18/TIM4_CH2/EVENTOUT)
- net OTG_CURRENT_LIMIT_SELECTION: now also U?.2 (PE3-TRACED0/FSMC_A19/EVENTOUT), R?.2
- net OTG_FS_VBUS: no longer C?.2
- net PA1: now also U?.24 (PA1-USART2_RTS/UART4_RX/ETH_RMII_REF_CLK/ETH_MII_RX_CLK/TIM5_CH2/TIMM2_CH2/EVENTOUT-ADC123_IN1)
- net PA2: now also U?.25 (PA2-USART2_TX/TIM5_CH3/TIM9_CH1/TIM2_CH3/ETH_MDIO/EVENTOUT-ADC123_IN2)
- net PA4: now also U?.29 (PA4-SPI1_NSS/SPI3_NSS/USART2_CK/DCMI_HSYNC/OTG_HS_SOF/I2S3_WS/EVENTOUT-ADC123_IN4/DAC1_OUT)
- net PA6: now also U?.31 (PA6-SPI1_MISO/TIM8_BKIN/TIM13_CH1/DCMI_PIXCLK/TIM3_CH1/TIM1_BKIN/EVENTOUT-ADC12_IN6)
- net PA7: now also U?.32 (PA7-SPI1_MOSI/TIM8_CH1N/TIM14_CH1/TIM3_CH2/ETH_MII_RX_DV/TIM1_CH1N/RMII_CRS_DV/EVENTOUT-ADC12_IN7)
- net PA8: now also U?.67 (PA8-MCO1/USART1_CK/TIM1_CH1/I2C3_SCL/OTG_FS_SOF/EVENTOUT)
- net PB10: now also U?.4 (IO3), U?.47 (PB10-SPI2_SCK/I2S2_CK/I2C2_SCL/USART3_TX/OTG_HS_ULPI_D3/ETH_MII_RX_ER/TIM2_CH3/EVENTOUT), R?.2
- net PB11: now also U?.48 (PB11-I2C2_SDA/USART3_RX/OTG_HS_ULPI_D4/ETH_RMII_TX_EN/ETH_MII_TX_EN/TIM2_CH4/EVENTOUT)
- net PB12: now also U?.51 (PB12-SPI2_NSS/I2S2_WS/I2C2_SMBA/USART3_CK/TIM1_BKIN/CAN2_RX/OTG_HS_ULPI_D5/ETH_RMII_TXD0/ETH_MII_TXD0/OTG_HS_ID/EVENTOUT)
- net PB13: now also U?.52 (PB13-SPI2_SCK/I2S2_CK/USART3_CTS/TIM1_CH1N/CAN2_TX/OTG_HS_ULPI_D6/ETH_RMII_TXD1/ETH_MII_TXD1/EVENTOUT-OTG_HS_VBUS)
- net PB5: now also U?.91 (PB5-I2C1_SMBA/CAN2_RX/OTG_HS_ULPI_D7/ETH_PPS_OUT/TIM3_CH2/SPI1_MOSI/SPI3_MOSI/DCMI_D10/I2S3_SD/EVENTOUT)
- net PC1: now also U?.16 (PC1-ETH_MDC/EVENTOUT-ADC123_IN11)
- net PC4: now also U?.33 (PC4-ETH_RMII_RX_D0/ETH_MII_RX_D0/EVENTOUT-ADC12_IN14)
- net PC5: now also U?.34 (PC5-ETH_RMII_RX_D1/ETH_MII_RX_D1/EVENTOUT-ADC12_IN15)
- net PC6: now also U?.63 (PC6-I2S2_MCK/TIM8_CH1/SDIO_D6/USART6_TX/DCMI_D0/TIM3_CH1/EVENTOUT)
- net PC7: now also U?.64 (PC7-I2S3_MCK/TIM8_CH2/SDIO_D7/USART6_RX/DCMI_D1/TIM3_CH2/EVENTOUT)
- net PD0: now also U?.81 (PD0-FSMC_D2/CAN1_RX/EVENTOUT)
- net PD1: now also U?.82 (PD1-FSMC_D3/CAN1_TX/EVENTOUT)
- net PD10: now also U?.57 (PD10-FSMC_D15/USART3_CK/EVENTOUT)
- net PD14: now also U?.61 (PD14-FSMC_D0/TIM4_CH3/EVENTOUT/EVENTOUT)
- net PD15: now also U?.62 (PD15-FSMC_D1/TIM4_CH4/EVENTOUT)
- net PD7: now also U?.88 (PD7-USART2_CK/FSMC_NE1/FSMC_NCE2/EVENTOUT)
- net PD8: now also U?.55 (PD8-FSMC_D13/USART3_TX/EVENTOUT)
- net PD9: now also U?.56 (PD9-FSMC_D14/USART3_RX/EVENTOUT)
- net PE0: now also U?.97 (PE0-TIM4_ETR/FSMC_NBL0/DCMI_D2/EVENTOUT), R?.2
- net PE1: now also U?.98 (PE1-FSMC_NBL1/DCMI_D3/EVENTOUT)
- net PE10: now also U?.41 (PE10-FSMC_D7/TIM1_CH2N/EVENTOUT)
- net PE11: now also U?.42 (PE11-FSMC_D8/TIM1_CH2/EVENTOUT)
- net PE12: now also U?.43 (PE12-FSMC_D9/TIM1_CH3N/EVENTOUT)
- net PE13: now also U?.44 (PE13-FSMC_D10/TIM1_CH3/EVENTOUT)
- net PE14: now also U?.45 (PE14-FSMC_D11/TIM1_CH4/EVENTOUT)
- net PE15: now also U?.46 (PE15-FSMC_D12/TIM1_BKIN/EVENTOUT)
- net PE7: now also U?.38 (PE7-FSMC_D4/TIM1_ETR/EVENTOUT)
- net PE8: now also U?.39 (PE8-FSMC_D5/TIM1_CH1N/EVENTOUT)
- net PE9: now also U?.40 (PE9-FSMC_D6/TIM1_CH1/EVENTOUT)
- net SD_CARD_INSERTED: now also R?.1; no longer U?.2 (PE3-TRACED0/FSMC_A19/EVENTOUT)
- net SYSTEM_LOAD: no longer R?.2
- net VDD: now also R?.2
- net USER_BUTTON: no longer names the net of R?.1, SW?.2, SW?.4
- net USER_BUTTON: now also R?.1; no longer U?.4 (IO3), U?.47 (PB10-SPI2_SCK/I2S2_CK/I2C2_SCL/USART3_TX/OTG_HS_ULPI_D3/ETH_MII_RX_ER/TIM2_CH3/EVENTOUT)
Other:
- note added: "<-- Pins to the expansion slot (65 TOTAL)"
- note added: "Charger status pin: Open drain charge status output to indicate various\ncharger operation. Connect to the pull up rail using pull-up resistor.\nLOW indicates charge in progress. HIGH indicates charge complete or\ncharge disabled. When any fault condition occurs, STAT pin blinks at 1Hz.\nPin is pulled high to SYSTEM_LOAD (3V5-4V2), but MCU's GPIO pins are 5V tolerant."
- note added: "I2C Slave address: 0x6B"
- note added: "If using over 5V power sources (17VDC max), remove\nzero ohm resistor to save the ARM's life!\n\nUSB (device mode) is still functioning, but OTG\ncannot be used.\n\n1uF cap's voltage rating should be at least 25V."
- note added: "Iinmax = (1V/Rilim)*530\n\nThe actual input current limit is the lower value between ILIM setting and\nregister setting (REG00[2:0]). For example, if the register setting is 111\nfor 3A, and ILIM has a 353Ω resistor to ground for 1.5A, the input current\nlimit is 1.5A. ILIM pin can be used to set the input current limit rather than\nthe register settings."
- note added: "PGND: On PCB layout, connect directly to\nground connection of input and output\ncapacitors of the charger. A single point\nconnection is recommended between\npower PGND and the analog GND near\nthe IC's PGND pin."
- note added: "SETC-SETP capacitance\nshould be approx. 220nF."
- note added: "The INT pin sends active low, 256us pulse to\nhost to report charger device status and fault."
- note removed: "<-- Pins to the expansion slot"
- note removed: "I2C Slave address: 0x6BH"
- note removed: "If using over 5V power sources (17VDC max), remove\nzero ohm resistor to save the ARM's life!\n\nUSB (device mode) is still functioning, but OTG\ncannot be used."
- note removed: "Iinmax = (1V/Rilim)*530\n\nThe actual input current limit is the lower value between ILIM setting and\n register setting (REG00[2:0]). For example, if the register setting is 111\nfor 3A, and ILIM has a 353Ω resistor to ground for 1.5A, the input current\nlimit is 1.5A. ILIM pin can be used to set the input current limit rather than\nthe register settings."
- moved on the sheet: C42, C?, D?, R?
