File: ruuvitracker_revb_kicad/ruuvitracker.sch (KiCad schematic (older format))
At the start: 156 parts, among them J1 USB_MICRO_B, P1 EXPANDER_1, P10 TP, P11 SPK_BEFORE_AMP, P12 TP, P13 BATT, P14 HOLE, P15 HOLE, P16 HOLE, P17 HOLE, P18 CONN_1, P19 PWR, P2 EXPANDER_2, P20 TP, P21 PWR_SW, P22 TP, P23 TP, P3 EXPANDER_3, P4 TP, P5 HAPTIC, P6 TP, P7 TP, P8 TP, P9 TP, Q1 MOSFET_P, Q2 MOSFET_P, SW1 PUSH_BUTTON, SW2 PUSH_BUTTON, U1 STM32F4XX_LQFP100, U10 DRV2603, U11 TPD4E004, U12 TPD4E004, U13 TPS737XX_SON8, U14 L3GD20, U15 LM4890M_MM, U16 MICROPHONE, U17 SN74AVC4T245_RSV, U18 M24M01, U2 SIM908, U3 BQ24190, U4 ADMP404, U5 LSM303DLHC, U6 TPD4E004, U7 TPD4E004, U8 MICROSD_SIM_COMBO, U9 TPD4E004, X1 4-26MHZ

Commit message: Add P-MOSTET to enable SYSTEM_LOAD only using pwr switch
Parts:
- added P24: TP, symbol TP
- added Q3: MOSFET_P, symbol MOSFET_P
- added R7: 330k, symbol R
- gave numbers to parts that had none: 4
Connections:
- net labels added: ENABLE_SYSTEM_LOAD
- net labels removed: SD_VDD
- wire segments 699 -> 608
Other:
- note added: "System load delivers all the current\n(up to 5A) for the system. Voltage\nnever drops below 3V5 (programmable)\nunless battery dies totally."
- note added: "To get good loop stability, the resonant\nfrequency of the output inductor and\noutput capacitor should be designed\nbetween 15kHz and 25kHz. With 2.2μH\ninductor, the typical output capacitor\nvalue is 20μF."
- note removed: "System load delivers all the current (up to 5A) for the system.\nVoltage never drops below 3V5 (programmable) unless battery dies totally."
- note removed: "To get good loop stability, the resonant frequency of the output inductor\nand output capacitor should be designed between 15kHz and 25kHz. With\n2.2μH inductor, the typical output capacitor value is 20μF."
- moved on the sheet: C18, FB2, J1, P12, P6, P7, P8, P9, RP3, U12

Commit message: Small mods
Other:
- note added: "P-MOSFET CSD25302Q2 (2x2mm SON-6) for example:\n\n* -5A continuous current\n* -20A pulse current\n* Vgs(th) = -0,65V typical\n* Drain to source leakage (Vgs=0V) = -1uA max\n* Rds (Vgs=-2V5, Ids=-3A) = 75mohm max"
- note added: "RevB (draft #003)"
- note removed: "RevB (draft #002)"
Changed lines of the file:
@@
-EESchema Schematic File Version 2  date Sat 29 Dec 2012 01:45:27 PM EET
+EESchema Schematic File Version 2  date Sat 29 Dec 2012 03:38:39 PM EET
 LIBS:power
 LIBS:device
@@
 Title "RuuviTracker"
 Date "29 dec 2012"
-Rev "RevB (draft#002)"
+Rev "RevB (draft#003)"
 Comp "RuuviTracker.fi / Lauri Jämsä / lauri.jamsa@ruuvipenkki.fi"
 Comment1 "Attribution-NonCommercial-ShareAlike 3.0 Unported (CC BY-NC-SA 3.0)"
@@
 Comment4 ""
 $EndDescr
+Text Notes 8950 17600 0    30   Italic 0
+P-MOSFET CSD25302Q2 (2x2mm SON-6) for example:\n\n* -5A continuous current\n* -20A pulse current\n* Vgs(th) = -0,65V typical\n* Drain to source leakage (Vgs=0V) = -1uA max\n* Rds (Vgs=-2V5, Ids=-3A) = 75mohm max
 Text Label 31400 7000 0    60   ~ 0
 3V3_FET_VDD
@@
 http://www.ruuvitracker.fi
 Text Notes 16500 2550 0    60   Italic 12
-RevB (draft #002)
+RevB (draft #003)
 Text Notes 15500 2250 0    120  Italic 24
 Open Source Tracking Solution

Commit message: Replace 26pin expander#1 with 26x2 expander
Parts:
- removed C47: 1u, symbol C
- removed P1: EXPANDER_1, symbol CONN_26
- removed P3: EXPANDER_3, symbol CONN_26
- added C47: 1u, symbol CP1
- added P1: EXPANDER_1, symbol CONN_26X2
- R47: value 4k7 -> 1k
- R51, R52, R7, R9: value 330k -> 47k
Connections:
- net labels added: CHG_SYS
- wire segments 608 -> 703
Other:
- note added: "47k resistor draws 70uA\nwhen FET is turned on."
- note added: "52 + 32 = 84 pins total"
- note removed: "26 + 32 + 26 = 84 pins total"
- note removed: "330k resistor draws 10uA\nwhen FET is turned on."

Commit message: Minor mods, PA9-PA12 available on expansion connector
Connections:
- net labels added: PA10, PA11, PA12, PA9
- wire segments 703 -> 604

Commit message: Replace 8xres arrays with 4xres arrays
Parts:
- removed RP1, RP2: 1M, symbol R_PACK8
- added RP1, RP2, RP5, RP6: 1M, symbol R_PACK4
Other:
- note added: "- Read current 1 mA, typical\n- Write current 2mA, typical\n- Standby current 3 uA, typical\n- Data retention >200 years\n- 4 million erase/write cycles\n- M24M01 = 128k x 8bit = 128 kbytes\n- SO8 (narrow, 150 mil width) or TSSOP8 (we use this one)"
- note removed: "- Read current 1 mA, typical\n- Write current 2mA, typical\n- Standby current 3 uA, typical\n- Data retention >200 years\n- 4 million erase/write cycles\n- M24M01 = 128k x 8bit = 128 kbytes\n- SO8 (150 mil width) or TSSOP8"
- moved on the sheet: C55

Commit message: Add charger diodes, ferrite to MEMS MIC's power etc.
Parts:
- removed R28: 0, symbol R
- removed R5: NA, symbol R
- added D4, D5: SCHOTTKY, symbol SCHOTTKY
- added FB3: FILTER, symbol FILTER
Connections:
- net 3V3_FET_VDD: now also FB3.1; no longer C2.1, U4.3 (VDD)
- net HIGH_VOLTAGE_VBUS: now also D4.1 (A)
- net OTG_FS_VBUS: now also D5.1 (A)
- net at C33.2, U3.1 (VBUS), U3.24 (VBUS): now also D4.2 (K), D5.2 (K)
- new net: C2.1, FB3.2, U4.3 (VDD)
Other:
- note added: "RevB (draft #004)"
- note removed: "RevB (draft #003)"

Commit message: Add zener and remove schottkys
Parts:
- removed D4, D5: SCHOTTKY, symbol SCHOTTKY
- added D4: 6V_ZENER, symbol ZENER
- added R5: 47k, symbol R
Connections:
- net GND: now also D4.1 (A)
- net HIGH_VOLTAGE_VBUS: now also C18.1, C33.2, FB2.2, P1.4 (P4), U12.6 (VCC), U3.1 (VBUS), U3.24 (VBUS), R5.1
- removed net OTG_FS_VBUS: C18.1, FB2.2, P1.4 (P4), P2.13 (P13), U1.68 (PA9-USART1_TX/TIM1_CH2/I2C3_SMBA/DCMI_D0/EVENTOUT-OTG_FS_VBUS), U12.6 (VCC)
- new net OTG_FS_VBUS_MCU: D4.2 (K), P2.13 (P13), R5.2, U1.68 (PA9-USART1_TX/TIM1_CH2/I2C3_SMBA/DCMI_D0/EVENTOUT-OTG_FS_VBUS)
Other:
- note added: "Max current @ 12V\nthrough series\nresistor = 255uA.\n\nuC's 5V tolerant\npins' absolute max\nvalue = Vdd + 4V."
- note added: "STM32F4's reference manual says:\nWhen HNP or SRP is enabled the VBUS sensing pin (PA9)\npin should be connected to VBUS. The VBUS input ensures\nthat valid VBUS levels are supplied by the charge pump during\nUSB operations. Any unforeseen VBUS voltage drop below the\nVBUS valid threshold (4.25 V) leads to an OTG interrupt triggered\nby the session end detected bit (SEDET bit in OTG_FS_GOTGINT).\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"
- note added: "The INT pin sends active\nlow, 256us pulse to host\nto report charger device\nstatus and fault."
- note removed: "The INT pin sends active low, 256us pulse to\nhost to report charger device status and fault."

Commit message: Remove GSM's MIC, fix GSM's audio amp circuitry, own voltage divider for high_voltage input
Parts:
- removed P11: SPK_BEFORE_AMP, symbol CONN_2
- removed U16: MICROPHONE, symbol MICROPHONE
- added C56, C57: 1u, symbol C
- added C58: 10n, symbol C
- added R10, R12, R16, R17: 22k, symbol R
Connections:
- net GSM_MIC2N is gone; now on net GND: U2.28 (MIC2N), U6.5 (IO4)
- net MEMS_MIC_OUTPUT is gone; now on net GSM_MIC2P: C1.1, P1.21 (P21), U1.26 (PA3-USART2_RX/TIM5_CH4/TIM9_CH2/TIM2_CH4/OTG_HS_ULPI_D0/ETH_MII_COL/EVENTOUT-ADC123_IN3)
- net 3V3_FET_VDD: now also FB3.2; no longer FB3.1
- net BATTERY_CELL: no longer RP6.2 (P2)
- net GND: now also C55.1, RP6.2 (P2), C58.2; no longer C55.2
- net GSM_SPK1N: now also C56.2; no longer U15.4 (-IN)
- net GSM_SPK1P: now also C57.1; no longer U15.3 (+IN)
- net HIGH_VOLTAGE_VBUS: now also RP5.1 (P1); no longer RP5.3 (P3)
- net SYSTEM_LOAD: now also C34.1, U15.6 (VDD)
- net VDD: no longer C34.1, U15.6 (VDD)
- net at C2.1, U4.3 (VDD): now also FB3.1; no longer FB3.2
- net at C41.1, U15.2 (BYPASS): now also R17.2
- net HIGH_VOLTAGE_VBUS_VMEAS: now reaches RP6.7 (R2), RP6.8 (R1)
- net HIGH_VOLTAGE_VBUS_VMEAS: now also C58.1
- net at RP5.2 (P2): now also RP5.3 (P3)
- net at RP5.7 (R2): now also RP5.8 (R1)
- net BATTERY_VOLTAGE_MEASUREMENT renamed BATTERY_CELL_VMEAS
- net BATTERY_CELL_VMEAS: now also C55.2; no longer C55.1
- net SPK_AMP_OUT1: no longer names the net of SP1.1, U15.5 (VO1)
- net SPK_AMP_OUT1: now also R10.1
- net SPK_AMP_OUT2: no longer names the net of SP1.2, U15.8 (VO2)
- new net: R12.1, R17.1, U15.3 (+IN)
- new net: R10.2, R16.2, U15.4 (-IN)
- new net: C57.2, R16.1
- new net: C56.1, R12.2
- no-connect marks 59 -> 55
Other:
- note added: "GSM's Loudspeaker"
- note added: "If over 5V power source is in use, USB (device mode)\nis still functioning, but OTG cannot be used.\n\nFor best performance, VBUS should be\ndecoupled to PGND with 1μF capacitance.\nCap's voltage rating should be at least 25V."
- note added: "Reference design: SIM908_Reference_Design_Guide_Application_V1.00"
- note added: "Route MIC's signal wires according\ndifferential signal design rules.\n\nFor multi-layers PCB, audio lines should be\nlayout in the middle layer, and keep ground\nlayer under audio layer."
- note added: "SIM908's microphone input channel can be\nconfigured to a single ended mode. In this\nmode, the MICN can be left open. The negative\nterminal of the microphone can be connected\nto GND.\n\nInput gain of the microphone on the GSM module should\nbe 0dB! AT-command to set up the gain is AT+CMIC."
- note added: "Texas Instruments LM4890MM/NOPB's (MSOP package) key features:\n\n- Power Output at 5V & 1% THD 1 W (typ.)\n- Power Output at 3V3 & 1% THD 400 mW(typ.)\n- Shutdown Current 0.1 uA(typ.)"
- note removed: "Electret Condenser Microphone"
- note removed: "GSM's Microphone"
- note removed: "GSM's Speaker"
- note removed: "If using over 5V power sources (17VDC max), remove\nzero ohm resistor to save the ARM's life!\n\nUSB (device mode) is still functioning, but OTG\ncannot be used.\n\nFor best performance, VBUS should be\ndecoupled to PGND with 1μF capacitance.\nCap's voltage rating should be at least 25V."
- note removed: "Route MIC's signal wires according\ndifferential signal design rules.\n\nFor multi-layers PCB, audio lines should be\nlayout in the middle layer, and keep ground\nlayer under audio layer.\n\nTrace width should be 6-8 mil.\n\nPlace ESD IC close to the microphone headers."
- note removed: "Texas Instruments LM4890MM/NOPB's (MSOP package) key features:\n\n- PSRR at 217Hz, VDD = 5V (Fig. 1) 62 dB (typ.)\n- Power Output at 5V & 1% THD 1 W (typ.)\n- Power Output at 3V3 & 1% THD 400 mW(typ.)\n- Shutdown Current 0.1 μA(typ.)"
- moved on the sheet: C1, C2, C32, C34, C41, C48, C49, FB3, R29, SP1, U15, U18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
